File: power.kicad_sch (KiCad schematic)
At the start: 25 parts, among them U7 AP63205WU, U8 AP63203WU

Commit message: update BOM
Parts:
- R15, R16: value 3k3 -> 1k5
- R17: value 3k3 -> 1k2
- R18: value 1k2 -> 680; Part Number RC0402FR-07560RL -> RC0402FR-07680RL
Changed lines of the file:
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@@
 		(fields_autoplaced yes)
 		(property "Reference" "R17"
-			(at 134.62 172.72 0)
+			(at 134.62 172.7199 0)
 			(effects
 				(font
@@
 			)
 		)
-		(property "Value" "3k3"
-			(at 134.62 175.26 0)
+		(property "Value" "1k2"
+			(at 134.62 175.2599 0)
 			(effects
 				(font
@@
 		(fields_autoplaced yes)
 		(property "Reference" "R18"
-			(at 153.67 172.72 0)
+			(at 153.67 172.7199 0)
 			(effects
 				(font
@@
 			)
 		)
-		(property "Value" "1k2"
-			(at 153.67 175.26 0)
+		(property "Value" "680"
+			(at 153.67 175.2599 0)
 			(effects
 				(font
@@
 			)
 		)
-		(property "Part Number" "RC0402FR-07560RL"
+		(property "Part Number" "RC0402FR-07680RL"
 			(at 151.13 173.99 0)
 			(effects
@@
 		(fields_autoplaced yes)
 		(property "Reference" "R15"
-			(at 87.63 172.72 0)
+			(at 87.63 172.7199 0)
 			(effects
 				(font
@@
 			)
 		)
-		(property "Value" "3k3"
-			(at 87.63 175.26 0)
+		(property "Value" "1k5"
+			(at 87.63 175.2599 0)
 			(effects
 				(font
@@
 		(fields_autoplaced yes)
 		(property "Reference" "R16"
-			(at 63.5 172.72 0)
+			(at 63.5 172.7199 0)
 			(effects
 				(font
@@
 			)
 		)
-		(property "Value" "3k3"
-			(at 63.5 175.26 0)
+		(property "Value" "1k5"
+			(at 63.5 175.2599 0)
 			(effects
 				(font
