File: untitled.kicad_sch (KiCad schematic)
At the start: 18 parts, among them U13 TJA1051TK-3, U14 TJA1051TK-3

Commit message: update BOM
Parts:
- U13, U14: Part Number (none) -> TJA1051TK-3
Changed lines of the file:
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@@
+			)
+		)
+		(property "Part Number" "TJA1051TK-3"
+			(at 154.94 128.27 0)
+			(effects
+				(font
+					(size 1.27 1.27)
+				)
+				(hide yes)
 			)
 		)
@@
 			(at 156.21 77.47 0)
 			(effects
+				(font
+					(size 1.27 1.27)
+				)
+				(hide yes)
+			)
+		)
+		(property "Part Number" "TJA1051TK-3"
+			(at 156.21 77.47 0)
+			(effects
