File: f405-fc-mcu_sch.kicad_sch (KiCad schematic)
At the start: 31 parts, among them SW1 SW_Push, U1 STM32F765VITx, Y1 16MHz

Commit message: use smaller button
Parts:
- SW1: footprint Project:SWITCH_EVQP2_PAN -> Project:EVPAA602
Changed lines of the file:
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@@
 			)
 		)
-		(property "Footprint" "Project:SWITCH_EVQP2_PAN"
+		(property "Footprint" "Project:EVPAA602"
 			(at 59.69 57.15 0)
 			(effects
